File: Rev. 1/Eagle/C64_AV-Adaptor.brd (EAGLE design)
At the start: 48 x 34 mm, 13 parts, among them J1 RTC9028, J2 SV80, J3 BTOR1 WHT, J4 BTOR1 RED, J5 BTOR1 BLK, J6 BTOR1 YE

Commit message: Silk Screen Update
Parts:
- added U$25: OPEN_SOURCE_HW, Logo:OPENHW
- moved U$23 26.7 mm to (20.0, 31.3)
Other:
- board text added: "330R"
- board text added: "Lumberg SV80"
- board text added: "blk"
- board text added: "http://github.com/ svenpetersen1965"
- board text added: "red"
- board text added: "wht"
- board text added: "yel"
